File: pcb/2364Adapter_v1.1.sch (EAGLE design)
At the start: 10 parts, among them IC1 2364, IC2 EPROM

Commit message: Added media
Parts:
- removed A13, A14, A15, GND: TPTP12R, testpad:TPTP12R
- added X1: (no value), con-lstb-rp:MA04-1
Connections:
- net A13: now also X1.4; no longer A13.TP
- net A14: now also X1.3; no longer A14.TP
- net A15: now also X1.2; no longer A15.TP
- net GND: now also X1.1; no longer GND.TP
Other:
- moved on the sheet: R1, R2, R3
Changed lines of the file:
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@@
 <part name="IC1" library="commodore" deviceset="2364" device="-RP" value="2364"/>
 <part name="GOLD_ORB_SM1" library="oshw" deviceset="OSHWLOGO" device="LOGO5MM" value="Open Source Hardware"/>
-<part name="A13" library="testpad" deviceset="TP" device="TP12R"/>
-<part name="A14" library="testpad" deviceset="TP" device="TP12R"/>
-<part name="A15" library="testpad" deviceset="TP" device="TP12R"/>
-<part name="GND" library="testpad" deviceset="TP" device="TP12R"/>
 <part name="SUPPLY3" library="supply2" deviceset="GND" device=""/>
+<part name="X1" library="con-lstb-rp" deviceset="MA04-1" device=""/>
 </parts>
 <sheets>
@@
 <instance part="FRAME1" gate="G$2" x="162.56" y="0"/>
 <instance part="SUPPLY1" gate="GND" x="53.34" y="50.8"/>
-<instance part="R1" gate="G$1" x="22.86" y="154.94" rot="R90"/>
-<instance part="R2" gate="G$1" x="27.94" y="154.94" rot="R90"/>
-<instance part="R3" gate="G$1" x="33.02" y="154.94" rot="R90"/>
-<instance part="SUPPLY2" gate="G$1" x="27.94" y="167.64"/>
+<instance part="R1" gate="G$1" x="20.32" y="154.94" rot="R90"/>
+<instance part="R2" gate="G$1" x="25.4" y="154.94" rot="R90"/>
+<instance part="R3" gate="G$1" x="30.48" y="154.94" rot="R90"/>
+<instance part="SUPPLY2" gate="G$1" x="25.4" y="167.64"/>
 <instance part="IC2" gate="G$1" x="68.58" y="86.36"/>
 <instance part="IC1" gate="G$1" x="68.58" y="139.7"/>
 <instance part="GOLD_ORB_SM1" gate="G$1" x="134.62" y="15.24"/>
-<instance part="A13" gate="G$1" x="27.94" y="137.16" smashed="yes" rot="R90">
-<attribute name="NAME" x="26.67" y="138.43" size="1.778" layer="95" rot="R180"/>
-<attribute name="TP_SIGNAL_NAME" x="29.21" y="138.43" size="1.778" layer="97" rot="R90"/>
-</instance>
-<instance part="A14" gate="G$1" x="27.94" y="134.62" smashed="yes" rot="R90">
-<attribute name="NAME" x="26.67" y="135.89" size="1.778" layer="95" rot="R180"/>
-<attribute name="TP_SIGNAL_NAME" x="29.21" y="135.89" size="1.778" layer="97" rot="R90"/>
-</instance>
-<instance part="A15" gate="G$1" x="27.94" y="132.08" smashed="yes" rot="R90">
-<attribute name="NAME" x="26.67" y="133.35" size="1.778" layer="95" rot="R180"/>
-<attribute name="TP_SIGNAL_NAME" x="29.21" y="133.35" size="1.778" layer="97" rot="R90"/>
-</instance>
-<instance part="GND" gate="G$1" x="27.94" y="129.54" smashed="yes" rot="R90">
-<attribute name="NAME" x="26.67" y="130.81" size="1.778" layer="95" rot="R180"/>
-<attribute name="TP_SIGNAL_NAME" x="29.21" y="130.81" size="1.778" layer="97" rot="R90"/>
-</instance>
-<instance part="SUPPLY3" gate="GND" x="38.1" y="121.92"/>
+<instance part="SUPPLY3" gate="GND" x="20.32" y="134.62"/>
+<instance part="X1" gate="1" x="10.16" y="144.78"/>
 </instances>
 <busses>
@@
 <net name="A13" class="0">
 <segment>
-<wire x1="40.64" y1="139.7" x2="38.1" y2="142.24" width="0.1524" layer="91"/>
-<wire x1="38.1" y1="142.24" x2="22.86" y2="142.24" width="0.1524" layer="91"/>
-<wire x1="22.86" y1="149.86" x2="22.86" y2="142.24" width="0.1524" layer="91"/>
-<label x="33.02" y="142.24" size="1.778" layer="95"/>
-<pinref part="R1" gate="G$1" pin="1"/>
-</segment>
-<segment>
 <wire x1="40.64" y1="71.12" x2="43.18" y2="73.66" width="0.1524" layer="91"/>
 <wire x1="43.18" y1="73.66" x2="55.88" y2="73.66" width="0.1524" layer="91"/>
@@
 </segment>
 <segment>
-<pinref part="A13" gate="G$1" pin="TP"/>
-<wire x1="40.64" y1="134.62" x2="38.1" y2="137.16" width="0.1524" layer="91"/>
-<wire x1="38.1" y1="137.16" x2="30.48" y2="137.16" width="0.1524" layer="91"/>
+<pinref part="X1" gate="1" pin="4"/>
+<wire x1="40.64" y1="144.78" x2="38.1" y2="147.32" width="0.1524" layer="91"/>
+<wire x1="38.1" y1="147.32" x2="20.32" y2="147.32" width="0.1524" layer="91"/>
+<wire x1="20.32" y1="149.86" x2="20.32" y2="147.32" width="0.1524" layer="91"/>
+<label x="38.1" y="142.24" size="1.778" layer="95" rot="MR0"/>
+<pinref part="R1" gate="G$1" pin="1"/>
+<wire x1="17.78" y1="147.32" x2="20.32" y2="147.32" width="0.1524" layer="91"/>
+<junction x="20.32" y="147.32"/>
 </segment>
 </net>
 <net name="A14" class="0">
-<segment>
-<wire x1="40.64" y1="142.24" x2="38.1" y2="144.78" width="0.1524" layer="91"/>
-<wire x1="38.1" y1="144.78" x2="27.94" y2="144.78" width="0.1524" layer="91"/>
-<wire x1="27.94" y1="149.86" x2="27.94" y2="144.78" width="0.1524" layer="91"/>
-<label x="33.02" y="144.78" size="1.778" layer="95"/>
-<pinref part="R2" gate="G$1" pin="1"/>
-</segment>
 <segment>
 <wire x1="40.64" y1="68.58" x2="43.18" y2="71.12" width="0.1524" layer="91"/>
@@
 </segment>
 <segment>
-<pinref part="A14" gate="G$1" pin="TP"/>
-<wire x1="40.64" y1="132.08" x2="38.1" y2="134.62" width="0.1524" layer="91"/>
-<wire x1="38.1" y1="134.62" x2="30.48" y2="134.62" width="0.1524" layer="91"/>
+<pinref part="X1" gate="1" pin="3"/>
+<wire x1="40.64" y1="142.24" x2="38.1" y2="144.78" width="0.1524" layer="91"/>
+<wire x1="38.1" y1="144.78" x2="25.4" y2="144.78" width="0.1524" layer="91"/>
+<wire x1="25.4" y1="149.86" x2="25.4" y2="144.78" width="0.1524" layer="91"/>
+<label x="38.1" y="144.78" size="1.778" layer="95" rot="MR0"/>
+<pinref part="R2" gate="G$1" pin="1"/>
+<wire x1="17.78" y1="144.78" x2="25.4" y2="144.78" width="0.1524" layer="91"/>
+<junction x="25.4" y="144.78"/>
 </segment>
 </net>
@@
 </segment>
 <segment>
-<pinref part="GND" gate="G$1" pin="TP"/>
-<wire x1="30.48" y1="129.54" x2="38.1" y2="129.54" width="0.1524" layer="91"/>
-<wire x1="38.1" y1="129.54" x2="38.1" y2="124.46" width="0.1524" layer="91"/>
+<wire x1="17.78" y1="139.7" x2="20.32" y2="139.7" width="0.1524" layer="91"/>
+<wire x1="20.32" y1="139.7" x2="20.32" y2="137.16" width="0.1524" layer="91"/>
 <pinref part="SUPPLY3" gate="GND" pin="GND"/>
+<pinref part="X1" gate="1" pin="1"/>
 </segment>
 </net>
 <net name="VCC" class="0">
 <segment>
-<wire x1="22.86" y1="160.02" x2="22.86" y2="162.56" width="0.1524" layer="91"/>
-<wire x1="22.86" y1="162.56" x2="27.94" y2="162.56" width="0.1524" layer="91"/>
-<wire x1="27.94" y1="162.56" x2="27.94" y2="160.02" width="0.1524" layer="91"/>
-<wire x1="27.94" y1="162.56" x2="33.02" y2="162.56" width="0.1524" layer="91"/>
-<wire x1="33.02" y1="162.56" x2="33.02" y2="160.02" width="0.1524" layer="91"/>
-<wire x1="27.94" y1="162.56" x2="27.94" y2="165.1" width="0.1524" layer="91"/>
-<junction x="27.94" y="162.56"/>
+<wire x1="20.32" y1="160.02" x2="20.32" y2="162.56" width="0.1524" layer="91"/>
+<wire x1="20.32" y1="162.56" x2="25.4" y2="162.56" width="0.1524" layer="91"/>
+<wire x1="25.4" y1="162.56" x2="25.4" y2="160.02" width="0.1524" layer="91"/>
+<wire x1="25.4" y1="162.56" x2="30.48" y2="162.56" width="0.1524" layer="91"/>
+<wire x1="30.48" y1="162.56" x2="30.48" y2="160.02" width="0.1524" layer="91"/>
+<wire x1="25.4" y1="162.56" x2="25.4" y2="165.1" width="0.1524" layer="91"/>
+<junction x="25.4" y="162.56"/>
 <pinref part="R1" gate="G$1" pin="2"/>
 <pinref part="R2" gate="G$1" pin="2"/>
@@
 <net name="A15" class="0">
 <segment>
-<wire x1="40.64" y1="144.78" x2="38.1" y2="147.32" width="0.1524" layer="91"/>
-<wire x1="38.1" y1="147.32" x2="33.02" y2="147.32" width="0.1524" layer="91"/>
-<wire x1="33.02" y1="147.32" x2="33.02" y2="149.86" width="0.1524" layer="91"/>
-<label x="33.02" y="147.32" size="1.778" layer="95"/>
-<pinref part="R3" gate="G$1" pin="1"/>
-</segment>
-<segment>
 <wire x1="40.64" y1="66.04" x2="43.18" y2="68.58" width="0.1524" layer="91"/>
 <wire x1="43.18" y1="68.58" x2="55.88" y2="68.58" width="0.1524" layer="91"/>
@@
 </segment>
 <segment>
-<pinref part="A15" gate="G$1" pin="TP"/>
-<wire x1="40.64" y1="129.54" x2="38.1" y2="132.08" width="0.1524" layer="91"/>
-<wire x1="38.1" y1="132.08" x2="30.48" y2="132.08" width="0.1524" layer="91"/>
-</segment>
-</net>
+<pinref part="X1" gate="1" pin="2"/>
+<wire x1="40.64" y1="139.7" x2="38.1" y2="142.24" width="0.1524" layer="91"/>
+<wire x1="38.1" y1="142.24" x2="30.48" y2="142.24" width="0.1524" layer="91"/>
+<wire x1="30.48" y1="142.24" x2="30.48" y2="149.86" width="0.1524" layer="91"/>
+<label x="38.1" y="147.32" size="1.778" layer="95" rot="MR0"/>
+<pinref part="R3" gate="G$1" pin="1"/>
+<wire x1="17.78" y1="142.24" x2="30.48" y2="142.24" width="0.1524" layer="91"/>
+<junction x="30.48" y="142.24"/>
+</segment>
+</net>
